File: eagle/FemtecTester/FemtecTester.sch (EAGLE design)
At the start: 50 parts, among them IC1 FT232RL, IC2 ATMEGA644A, K1 AQY212, K2 AQY212

Commit message: update FemtoTester eagle files (rev. B)
Parts:
- K1, K2: device relay:AQY21SOP -> tpv:AQY2212VEHA
Other:
- moved on the sheet: LED-5, LED-6, R7, R8
Changed lines of the file:
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@@
 <?xml version="1.0" encoding="utf-8"?>
 <!DOCTYPE eagle SYSTEM "eagle.dtd">
-<eagle version="6.4">
+<eagle version="6.5.0">
 <drawing>
 <settings>
@@
 <part name="LED-5" library="led" deviceset="LED" device="CHIPLED_1206" value="red"/>
 <part name="GND14" library="supply1" deviceset="GND" device=""/>
-<part name="K1" library="relay" deviceset="AQY*" device="SOP" technology="21" value="AQY212"/>
-<part name="K2" library="relay" deviceset="AQY*" device="SOP" technology="21" value="AQY212"/>
+<part name="K1" library="tpv" deviceset="AQY221*2V" device="EHA" value="AQY212"/>
+<part name="K2" library="tpv" deviceset="AQY221*2V" device="EHA" value="AQY212"/>
 <part name="FS" library="con-molex" deviceset="22-?-04" device="05-7048"/>
 <part name="R9" library="rcl" deviceset="R-EU_" device="M1206" value="750"/>
@@
 <attribute name="VALUE" x="33.655" y="140.208" size="1.778" layer="96" rot="R90"/>
 </instance>
-<instance part="LED-6" gate="G$1" x="137.16" y="58.42" smashed="yes">
-<attribute name="NAME" x="140.716" y="53.848" size="1.778" layer="95" rot="R90"/>
-<attribute name="VALUE" x="135.255" y="58.928" size="1.778" layer="96" rot="R90"/>
+<instance part="LED-6" gate="G$1" x="139.7" y="58.42" smashed="yes">
+<attribute name="NAME" x="143.256" y="53.848" size="1.778" layer="95" rot="R90"/>
+<attribute name="VALUE" x="137.795" y="58.928" size="1.778" layer="96" rot="R90"/>
 </instance>
 <instance part="R1" gate="G$1" x="241.3" y="88.9" rot="R180"/>
@@
 <instance part="R6" gate="G$1" x="12.7" y="149.86" rot="R270"/>
 <instance part="GND13" gate="1" x="12.7" y="124.46"/>
-<instance part="R7" gate="G$1" x="137.16" y="68.58" rot="R90"/>
-<instance part="R8" gate="G$1" x="144.78" y="68.58" rot="R90"/>
-<instance part="LED-5" gate="G$1" x="144.78" y="58.42" smashed="yes">
-<attribute name="NAME" x="148.336" y="53.848" size="1.778" layer="95" rot="R90"/>
-<attribute name="VALUE" x="142.875" y="58.928" size="1.778" layer="96" rot="R90"/>
+<instance part="R7" gate="G$1" x="139.7" y="68.58" rot="R90"/>
+<instance part="R8" gate="G$1" x="147.32" y="68.58" rot="R90"/>
+<instance part="LED-5" gate="G$1" x="147.32" y="58.42" smashed="yes">
+<attribute name="NAME" x="150.876" y="53.848" size="1.778" layer="95" rot="R90"/>
+<attribute name="VALUE" x="145.415" y="58.928" size="1.778" layer="96" rot="R90"/>
 </instance>
-<instance part="GND14" gate="1" x="144.78" y="45.72"/>
+<instance part="GND14" gate="1" x="147.32" y="45.72"/>
 <instance part="K1" gate="G$1" x="137.16" y="30.48"/>
 <instance part="K2" gate="G$1" x="137.16" y="15.24"/>
@@
 </segment>
 </bus>
-<bus name="RX,TX,CTS,DTS">
+<bus name="RX,TX,CTS,DTS,DTR">
 <segment>
 <wire x1="121.92" y1="43.18" x2="121.92" y2="55.88" width="0.762" layer="92"/>
@@
 <pinref part="LED-5" gate="G$1" pin="C"/>
 <pinref part="GND14" gate="1" pin="GND"/>
-<wire x1="144.78" y1="53.34" x2="144.78" y2="50.8" width="0.1524" layer="91"/>
+<wire x1="147.32" y1="53.34" x2="147.32" y2="50.8" width="0.1524" layer="91"/>
 <pinref part="LED-6" gate="G$1" pin="C"/>
-<wire x1="144.78" y1="50.8" x2="144.78" y2="48.26" width="0.1524" layer="91"/>
-<wire x1="137.16" y1="53.34" x2="137.16" y2="50.8" width="0.1524" layer="91"/>
-<wire x1="137.16" y1="50.8" x2="144.78" y2="50.8" width="0.1524" layer="91"/>
-<junction x="144.78" y="50.8"/>
+<wire x1="147.32" y1="50.8" x2="147.32" y2="48.26" width="0.1524" layer="91"/>
+<wire x1="139.7" y1="53.34" x2="139.7" y2="50.8" width="0.1524" layer="91"/>
+<wire x1="139.7" y1="50.8" x2="147.32" y2="50.8" width="0.1524" layer="91"/>
+<junction x="147.32" y="50.8"/>
 </segment>
 <segment>
@@
 <pinref part="R7" gate="G$1" pin="1"/>
 <pinref part="LED-6" gate="G$1" pin="A"/>
-<wire x1="137.16" y1="63.5" x2="137.16" y2="60.96" width="0.1524" layer="91"/>
+<wire x1="139.7" y1="63.5" x2="139.7" y2="60.96" width="0.1524" layer="91"/>
 </segment>
 </net>
@@
 <pinref part="R8" gate="G$1" pin="1"/>
 <pinref part="LED-5" gate="G$1" pin="A"/>
-<wire x1="144.78" y1="63.5" x2="144.78" y2="60.96" width="0.1524" layer="91"/>
+<wire x1="147.32" y1="63.5" x2="147.32" y2="60.96" width="0.1524" layer="91"/>
 </segment>
 </net>
@@
 <segment>
 <pinref part="IC2" gate="G$1" pin="(PCINT22/TOSC1)PC6"/>
-<wire x1="104.14" y1="76.2" x2="137.16" y2="76.2" width="0.1524" layer="91"/>
+<wire x1="104.14" y1="76.2" x2="139.7" y2="76.2" width="0.1524" layer="91"/>
 <pinref part="R7" gate="G$1" pin="2"/>
-<wire x1="137.16" y1="76.2" x2="137.16" y2="73.66" width="0.1524" layer="91"/>
+<wire x1="139.7" y1="76.2" x2="139.7" y2="73.66" width="0.1524" layer="91"/>
+<label x="134.62" y="73.66" size="1.778" layer="95"/>
 </segment>
 </net>
@@
 <segment>
 <pinref part="IC2" gate="G$1" pin="(PCINT23/TOSC2)PC7"/>
-<wire x1="104.14" y1="78.74" x2="144.78" y2="78.74" width="0.1524" layer="91"/>
+<wire x1="104.14" y1="78.74" x2="147.32" y2="78.74" width="0.1524" layer="91"/>
 <pinref part="R8" gate="G$1" pin="2"/>
-<wire x1="144.78" y1="78.74" x2="144.78" y2="73.66" width="0.1524" layer="91"/>
-</segment>
-</net>
+<wire x1="147.32" y1="78.74" x2="147.32" y2="73.66" width="0.1524" layer="91"/>
+<label x="134.62" y="78.74" size="1.778" layer="95"/>
+</segment>
+</net>
